File: Electronics/ThermoSanitizer.sch (KiCad schematic (older format))
At the start: 12 parts

Commit message: edit pcb
Parts:
- removed J?: I/O, symbol Connector:Conn_01x06_Female
- removed U?: ATtiny85-20SU, Package_SO:SOIJ-8_5.3x5.3mm_P1.27mm, symbol MCU_Microchip_ATtiny:ATtiny85-20SU
- added A?: Arduino_Nano_v3.x, Module:Arduino_Nano, symbol MCU_Module:Arduino_Nano_v3.x
- added C?: 0,1uf, symbol Device:C_Small
- added D? (x2): 1N5400, Diode_THT:D_DO-201AD_P15.24mm_Horizontal, symbol Diode:1N5400
- added J?: I2C, symbol Connector:Conn_01x04_Male
- added J?: Motor_OUT, symbol Connector:Conn_01x02_Male
- added Q?: IRF540N, Package_TO_SOT_THT:TO-220-3_Vertical, symbol Transistor_FET:IRF540N
- added R?: 1K, symbol Device:R_Small
- C?: value 0,1uf -> 4,7
- C?: value 4,7uf -> 1uf
Connections:
- net +5V: now also A?.30 (VIN), C?.1, D?.1 (K), J?.1 (Pin_1), J?.2 (Pin_2)
- net +BATT: now also D?.2 (A); no longer C?.1, U?.1 (IN)
- net GND: now also A?.29 (GND), A?.4 (GND), C?.2, J?.4 (Pin_4), Q?.3 (S), R?.2
- net SCL: now also A?.24 (A5), J?.3 (Pin_3)
- net SDA: now also A?.23 (A4), J?.2 (Pin_2)
- net TRIG&ECHO: now also A?.9 (D6)
- new net: C?.1, D?.1 (K), U?.1 (IN)
- new net: D?.2 (A), J?.1 (Pin_1), Q?.2 (D)
- new net MOTOR: A?.12 (D9), Q?.1 (G), R?.1
Other:
- moved on the sheet: C?, J?, U?

Commit message: add invoice and canva project
Parts:
- removed J?: Batt, symbol Connector:Conn_01x02_Male
- removed J?: Motor_OUT, symbol Connector:Conn_01x02_Male
- added H1, H2, H3, H4: MountingHole_Pad, MountingHole:MountingHole_3.2mm_M3, symbol Mechanical:MountingHole_Pad
- added J2: Barrel_Jack, Connector_BarrelJack:BarrelJack_Horizontal, symbol Connector:Barrel_Jack
- added J5: Motor_Out, Connector_PinHeader_2.54mm:PinHeader_1x02_P2.54mm_Vertical, symbol Connector:Screw_Terminal_01x02
- C1: renamed from C?; value 4,7uf -> 4,7uF; footprint (none) -> Capacitor_THT:C_Disc_D7.5mm_W5.0mm_P7.50mm
- C2, C5: renamed from C?; value 0,1uf -> 0,1uF; footprint (none) -> Capacitor_THT:C_Disc_D7.5mm_W5.0mm_P7.50mm
- C3: renamed from C?; value 1uf -> 1uF; footprint (none) -> Capacitor_THT:C_Disc_D7.5mm_W5.0mm_P7.50mm
- C4: renamed from C?; value 4,7 -> 4,7uF; footprint (none) -> Capacitor_THT:C_Disc_D7.5mm_W5.0mm_P7.50mm
- D1: renamed from D?; footprint (none) -> LED_THT:LED_D5.0mm
- J1: renamed from J?; footprint (none) -> Connector_PinHeader_2.54mm:PinHeader_1x02_P2.54mm_Vertical
- J3, J4: renamed from J?; footprint (none) -> Connector_PinSocket_2.54mm:PinSocket_1x04_P2.54mm_Horizontal
- R1, R2: renamed from R?; footprint (none) -> Resistor_THT:R_Axial_DIN0207_L6.3mm_D2.5mm_P2.54mm_Vertical
- U1: renamed from U?; footprint (none) -> Package_TO_SOT_THT:TO-220-2_Horizontal_TabDown
- gave numbers to parts that had none: 4
Connections:
- net +5V: now also J5.1 (Pin_1)
- net GND: now also H1.1, H2.1, H3.1, H4.1, J2.2
- net MOTOR: now also A1.8 (D5); no longer A1.12 (D9)
- net TRIG&ECHO: now also A1.13 (D10); no longer A1.9 (D6)
- net at D3.2 (A), Q1.2 (D): now also J5.2 (Pin_2)
- net +BATT renamed VBUS
- net VBUS: now also J2.1
Other:
- note added: "Arduino"
- note added: "Connectors"
- note added: "Decoupling Caps"
- note added: "LED Indicator"
- note added: "Motor Driver"
- note added: "Mounting Hole"
- note added: "Voltage Regulator"
- moved on the sheet: A1, C1, C2, C3, C4, C5, D1, D2, D3, J1, J3, J4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
