File: ThermoSanitizer Electronics/ThermoSanitizer.sch (KiCad schematic (older format))
At the start: 22 parts, among them J1 5V_Thermo, J3 Ultrasonic, J4 I2C, J5 Motor_Out, Q1 IRF540N, U1 L7805

Commit message: add clock switch
Parts:
- removed C1: 4,7uF, Capacitor_THT:C_Disc_D7.5mm_W5.0mm_P7.50mm, symbol Device:C_Small
- removed C2: 0,1uF, Capacitor_THT:C_Disc_D7.5mm_W5.0mm_P7.50mm, symbol Device:C_Small
- removed D1: LED, LED_THT:LED_D5.0mm, symbol Device:LED
- removed J1: 5V_Thermo, Connector_PinHeader_2.54mm:PinHeader_1x02_P2.54mm_Vertical, symbol Connector:Conn_01x02_Male
- removed J4: I2C, Connector_PinSocket_2.54mm:PinSocket_1x04_P2.54mm_Horizontal, symbol Connector:Conn_01x04_Male
- removed J?: Barrel_Jack, symbol Connector:Barrel_Jack
- removed R1: 120R, Resistor_THT:R_Axial_DIN0207_L6.3mm_D2.5mm_P2.54mm_Vertical, symbol Device:R_Small
- added J1: 5V_Thermo, TerminalBlock:TerminalBlock_bornier-2_P5.08mm, symbol Connector:Screw_Terminal_01x02
- added J2: 9V_In, TerminalBlock:TerminalBlock_bornier-2_P5.08mm, symbol Connector:Screw_Terminal_01x02
- C3: value 1uF -> 10uF
- C4: value 4,7uF -> 0.1uF
- C5: value 0,1uF -> 1uF
- J5: footprint Connector_PinHeader_2.54mm:PinHeader_1x02_P2.54mm_Vertical -> TerminalBlock:TerminalBlock_bornier-2_P5.08mm
- U1: footprint Package_TO_SOT_THT:TO-220-2_Horizontal_TabDown -> Package_TO_SOT_THT:TO-220-3_Vertical
Connections:
- net labels added: +9V
- net labels removed: VBUS
- wire segments 64 -> 52
Other:
- note removed: "Decoupling Caps"
- note removed: "LED Indicator"
Changed lines of the file:
@@
-$EndComp
-$Comp
-L Connector:Conn_01x02_Male J1
-U 1 1 60F8BE49
-P 6900 2550
-F 0 "J1" H 7008 2731 50  0000 C CNN
-F 1 "5V_Thermo" H 7008 2640 50  0000 C CNN
-F 2 "Connector_PinHeader_2.54mm:PinHeader_1x02_P2.54mm_Vertical" H 6900 2550 50  0001 C CNN
-F 3 "~" H 6900 2550 50  0001 C CNN
-	1    6900 2550
-	1    0    0    -1
 $EndComp
 $Comp
@@
 TRIG&ECHO
 $Comp
-L Device:C_Small C1
-U 1 1 60F93440
-P 3050 1200
-F 0 "C1" H 3142 1246 50  0000 L CNN
-F 1 "4,7uF" H 3142 1155 50  0000 L CNN
-F 2 "Capacitor_THT:C_Disc_D7.5mm_W5.0mm_P7.50mm" H 3050 1200 50  0001 C CNN
-F 3 "~" H 3050 1200 50  0001 C CNN
-	1    3050 1200
-	1    0    0    -1
-$EndComp
-$Comp
-L Device:C_Small C2
-U 1 1 60F93E00
-P 3450 1200
-F 0 "C2" H 3542 1246 50  0000 L CNN
-F 1 "0,1uF" H 3542 1155 50  0000 L CNN
-F 2 "Capacitor_THT:C_Disc_D7.5mm_W5.0mm_P7.50mm" H 3450 1200 50  0001 C CNN
-F 3 "~" H 3450 1200 50  0001 C CNN
-	1    3450 1200
-	1    0    0    -1
-$EndComp
-$Comp
-L power:GND #PWR02
-U 1 1 60F94D5C
-P 3450 1450
-F 0 "#PWR02" H 3450 1200 50  0001 C CNN
-F 1 "GND" H 3455 1277 50  0000 C CNN
-F 2 "" H 3450 1450 50  0001 C CNN
-F 3 "" H 3450 1450 50  0001 C CNN
-	1    3450 1450
-	1    0    0    -1
-$EndComp
-$Comp
-L power:+5V #PWR01
-U 1 1 60F95D6F
-P 3450 900
-F 0 "#PWR01" H 3450 750 50  0001 C CNN
-F 1 "+5V" H 3465 1073 50  0000 C CNN
-F 2 "" H 3450 900 50  0001 C CNN
-F 3 "" H 3450 900 50  0001 C CNN
-	1    3450 900
-	1    0    0    -1
-$EndComp
-Wire Wire Line
-	3450 1100 3050 1100
-Wire Wire Line
-	3450 1300 3050 1300
-Wire Wire Line
-	3450 1450 3450 1300
-Connection ~ 3450 1300
-Wire Wire Line
-	3450 1100 3450 900
-Connection ~ 3450 1100
-$Comp
-L Device:LED D1
-U 1 1 60F98123
-P 3450 2350
-F 0 "D1" V 3489 2232 50  0000 R CNN
-F 1 "LED" V 3398 2232 50  0000 R CNN
-F 2 "LED_THT:LED_D5.0mm" H 3450 2350 50  0001 C CNN
-F 3 "~" H 3450 2350 50  0001 C CNN
-	1    3450 2350
-	0    -1   -1   0
-$EndComp
-$Comp
-L power:+5V #PWR07
-U 1 1 60F99B96
-P 3450 2150
-F 0 "#PWR07" H 3450 2000 50  0001 C CNN
-F 1 "+5V" H 3465 2323 50  0000 C CNN
-F 2 "" H 3450 2150 50  0001 C CNN
-F 3 "" H 3450 2150 50  0001 C CNN
-	1    3450 2150
-	1    0    0    -1
-$EndComp
-$Comp
-L Device:R_Small R1
-U 1 1 60F9A719
-P 3450 2650
-F 0 "R1" H 3509 2696 50  0000 L CNN
-F 1 "120R" H 3509 2605 50  0000 L CNN
-F 2 "Resistor_THT:R_Axial_DIN0207_L6.3mm_D2.5mm_P2.54mm_Vertical" H 3450 2650 50  0001 C CNN
-F 3 "~" H 3450 2650 50  0001 C CNN
-	1    3450 2650
-	1    0    0    -1
-$EndComp
-$Comp
-L power:GND #PWR08
-U 1 1 60F9BCE3
-P 3450 2800
-F 0 "#PWR08" H 3450 2550 50  0001 C CNN
-F 1 "GND" H 3455 2627 50  0000 C CNN
-F 2 "" H 3450 2800 50  0001 C CNN
-F 3 "" H 3450 2800 50  0001 C CNN
-	1    3450 2800
-	1    0    0    -1
-$EndComp
-Wire Wire Line
-	3450 2200 3450 2150
-Wire Wire Line
-	3450 2550 3450 2500
-Wire Wire Line
-	3450 2800 3450 2750
-$Comp
 L Regulator_Linear:L7805 U1
 U 1 1 60F9E9C8
@@
 F 0 "U1" H 5250 2842 50  0000 C CNN
 F 1 "L7805" H 5250 2751 50  0000 C CNN
-F 2 "Package_TO_SOT_THT:TO-220-2_Horizontal_TabDown" H 5275 2450 50  0001 L CIN
+F 2 "Package_TO_SOT_THT:TO-220-3_Vertical" H 5275 2450 50  0001 L CIN
 F 3 "http://www.st.com/content/ccc/resource/technical/document/datasheet/41/4f/b3/b0/12/d4/47/88/CD00000444.pdf/files/CD00000444.pdf/jcr:content/translations/en.CD00000444.pdf" H 5250 2550 50  0001 C CNN
 	1    5250 2600
@@
 P 5650 2700
 F 0 "C4" H 5742 2746 50  0000 L CNN
-F 1 "4,7uF" H 5742 2655 50  0000 L CNN
+F 1 "0.1uF" H 5742 2655 50  0000 L CNN
 F 2 "Capacitor_THT:C_Disc_D7.5mm_W5.0mm_P7.50mm" H 5650 2700 50  0001 C CNN
 F 3 "~" H 5650 2700 50  0001 C CNN
@@
 L power:GND #PWR06
 U 1 1 60FA8FD5
-P 10850 2800
-F 0 "#PWR06" H 10850 2550 50  0001 C CNN
-F 1 "GND" H 10855 2627 50  0000 C CNN
-F 2 "" H 10850 2800 50  0001 C CNN
-F 3 "" H 10850 2800 50  0001 C CNN
-	1    10850 2800
+P 9850 2700
+F 0 "#PWR06" H 9850 2450 50  0001 C CNN
+F 1 "GND" H 9855 2527 50  0000 C CNN
+F 2 "" H 9850 2700 50  0001 C CNN
+F 3 "" H 9850 2700 50  0001 C CNN
+	1    9850 2700
 	1    0    0    -1
 $EndComp
@@
 P 4750 2700
 F 0 "C3" H 4842 2746 50  0000 L CNN
-F 1 "1uF" H 4842 2655 50  0000 L CNN
+F 1 "10uF" H 4842 2655 50  0000 L CNN
 F 2 "Capacitor_THT:C_Disc_D7.5mm_W5.0mm_P7.50mm" H 4750 2700 50  0001 C CNN
 F 3 "~" H 4750 2700 50  0001 C CNN
@@
 	4400 2600 4250 2600
 $Comp
-L Connector:Conn_01x04_Male J4
-U 1 1 60FDDF8B
-P 9150 2600
-F 0 "J4" H 9258 2881 50  0000 C CNN
-F 1 "I2C" H 9258 2790 50  0000 C CNN
-F 2 "Connector_PinSocket_2.54mm:PinSocket_1x04_P2.54mm_Horizontal" H 9150 2600 50  0001 C CNN
-F 3 "~" H 9150 2600 50  0001 C CNN
-	1    9150 2600
-	1    0    0    -1
-$EndComp
-$Comp
-L power:+5V #PWR015
-U 1 1 60FE07DC
-P 9750 2500
-F 0 "#PWR015" H 9750 2350 50  0001 C CNN
-F 1 "+5V" H 9765 2673 50  0000 C CNN
-F 2 "" H 9750 2500 50  0001 C CNN
-F 3 "" H 9750 2500 50  0001 C CNN
-	1    9750 2500
-	1    0    0    -1
-$EndComp
-$Comp
-L power:GND #PWR016
-U 1 1 60FE15C4
-P 9750 2850
-F 0 "#PWR016" H 9750 2600 50  0001 C CNN
-F 1 "GND" H 9755 2677 50  0000 C CNN
-F 2 "" H 9750 2850 50  0001 C CNN
-F 3 "" H 9750 2850 50  0001 C CNN
-	1    9750 2850
-	1    0    0    -1
-$EndComp
-Wire Wire Line
-	9750 2500 9350 2500
-Wire Wire Line
-	9750 2850 9750 2800
-Wire Wire Line
-	9750 2800 9350 2800
-Text GLabel 9650 2600 2    50   Input ~ 0
-SDA
-Wire Wire Line
-	9350 2600 9650 2600
-Text GLabel 9650 2700 2    50   Input ~ 0
-SCL
-Wire Wire Line
-	9350 2700 9650 2700
-$Comp
 L Device:C_Small C5
 U 1 1 60FEEE84
 P 6050 2700
 F 0 "C5" H 6142 2746 50  0000 L CNN
-F 1 "0,1uF" H 6142 2655 50  0000 L CNN
+F 1 "1uF" H 6142 2655 50  0000 L CNN
 F 2 "Capacitor_THT:C_Disc_D7.5mm_W5.0mm_P7.50mm" H 6050 2700 50  0001 C CNN
 F 3 "~" H 6050 2700 50  0001 C CNN
@@
 F 0 "J5" H 6130 892 50  0000 L CNN
 F 1 "Motor_Out" H 6130 801 50  0000 L CNN
-F 2 "Connector_PinHeader_2.54mm:PinHeader_1x02_P2.54mm_Vertical" H 6050 900 50  0001 C CNN
+F 2 "TerminalBlock:TerminalBlock_bornier-2_P5.08mm" H 6050 900 50  0001 C CNN
 F 3 "~" H 6050 900 50  0001 C CNN
 	1    6050 900
@@
 Arduino
 Wire Notes Line
-	2800 1850 4000 1850
-Text Notes 2950 1800 0    50   ~ 0
-Decoupling Caps
-Wire Notes Line
 	4000 500  4000 3300
-Text Notes 2950 3200 0    50   ~ 0
-LED Indicator
 Text Notes 4300 2100 0    50   ~ 0
 Motor Driver
@@
 Wire Notes Line
 	7900 2200 7900 500
-$Comp
-L power:VBUS #PWR09
-U 1 1 61033CBE
-P 10850 2600
-F 0 "#PWR09" H 10850 2450 50  0001 C CNN
-F 1 "VBUS" H 10865 2773 50  0000 C CNN
-F 2 "" H 10850 2600 50  0001 C CNN
-F 3 "" H 10850 2600 50  0001 C CNN
-	1    10850 2600
-	1    0    0    -1
-$EndComp
-$Comp
-L power:VBUS #PWR05
-U 1 1 610363C6
+Wire Wire Line
+	9700 2600 9850 2600
+Wire Wire Line
+	9850 2700 9700 2700
+$Comp
+L power:+9V #PWR02
+U 1 1 610EDB32
+P 9850 2600
+F 0 "#PWR02" H 9850 2450 50  0001 C CNN
+F 1 "+9V" H 9865 2773 50  0000 C CNN
+F 2 "" H 9850 2600 50  0001 C CNN
+F 3 "" H 9850 2600 50  0001 C CNN
+	1    9850 2600
+	1    0    0    -1
+$EndComp
+$Comp
+L Connector:Screw_Terminal_01x02 J2
+U 1 1 610F148C
+P 9500 2600
+F 0 "J2" H 9418 2817 50  0000 C CNN
+F 1 "9V_In" H 9418 2726 50  0000 C CNN
+F 2 "TerminalBlock:TerminalBlock_bornier-2_P5.08mm" H 9500 2600 50  0001 C CNN
+F 3 "~" H 9500 2600 50  0001 C CNN
+	1    9500 2600
+	-1   0    0    -1
+$EndComp
+$Comp
+L Connector:Screw_Terminal_01x02 J1
+U 1 1 610F3A6D
+P 6900 2550
+F 0 "J1" H 6818 2767 50  0000 C CNN
+F 1 "5V_Thermo" H 6818 2676 50  0000 C CNN
+F 2 "TerminalBlock:TerminalBlock_bornier-2_P5.08mm" H 6900 2550 50  0001 C CNN
+F 3 "~" H 6900 2550 50  0001 C CNN
+	1    6900 2550
+	-1   0    0    -1
+$EndComp
+$Comp
+L power:+9V #PWR01
+U 1 1 610F4CD8
 P 4250 2600
-F 0 "#PWR05" H 4250 2450 50  0001 C CNN
-F 1 "VBUS" H 4265 2773 50  0000 C CNN
+F 0 "#PWR01" H 4250 2450 50  0001 C CNN
+F 1 "+9V" H 4265 2773 50  0000 C CNN
 F 2 "" H 4250 2600 50  0001 C CNN
 F 3 "" H 4250 2600 50  0001 C CNN
@@
 	1    0    0    -1
 $EndComp
-$Comp
-L Connector:Barrel_Jack J?
-U 1 1 6104623D
-P 10450 2700
-F 0 "J?" H 10507 3025 50  0000 C CNN
-F 1 "Barrel_Jack" H 10507 2934 50  0000 C CNN
-F 2 "" H 10500 2660 50  0001 C CNN
-F 3 "~" H 10500 2660 50  0001 C CNN
-	1    10450 2700
-	1    0    0    -1
-$EndComp
-Wire Wire Line
-	10850 2600 10750 2600
-Wire Wire Line
-	10850 2800 10750 2800
 $EndSCHEMATC

Commit message: Adding alot of stuff
Parts:
- removed C3: 10uF, Capacitor_THT:C_Disc_D7.5mm_W5.0mm_P7.50mm, symbol Device:C_Small
- removed C4: 0.1uF, Capacitor_THT:C_Disc_D7.5mm_W5.0mm_P7.50mm, symbol Device:C_Small
- removed C5: 1uF, Capacitor_THT:C_Disc_D7.5mm_W5.0mm_P7.50mm, symbol Device:C_Small
- removed D2: 1N5400, Diode_THT:D_DO-201AD_P15.24mm_Horizontal, symbol Diode:1N5400
- removed H1, H2, H3, H4: MountingHole_Pad, MountingHole:MountingHole_3.2mm_M3, symbol Mechanical:MountingHole_Pad
- removed U1: L7805, Package_TO_SOT_THT:TO-220-3_Vertical, symbol Regulator_Linear:L7805
- added H1, H2, H3, H4: MountingHole, MountingHole:MountingHole_3.2mm_M3, symbol Mechanical:MountingHole
- renumbered D3 to D1, J3 to J1, J1 to J2, J2 to J3, J5 to J4, R2 to R1
Connections:
- net +5V: now also A1.27 (+5V); no longer A1.30 (VIN)
- net +9V: now also A1.30 (VIN)
- net SCL: no longer names the net of A1.24 (A5)
- net SDA: no longer names the net of A1.23 (A4)
- no-connect marks 0 -> 24
Other:
- note added: "Note: This project can be shrinked more with digispark, but I got no time left."
- note removed: "Voltage Regulator"
- moved on the sheet: J1, J2, J3
